Commit message: update

File: src/robot_description/urdf/my-robot.xacro (robot description, xacro)
@@ -2,10 +2,4 @@
 <robot xmlns:xacro="http://www.ros.org/wiki/xacro" name="robot">
     <xacro:property name="M_PI" value="3.14159"/>
-    <link name="world"/>
-    <joint name="joint_world" type="fixed">
-        <origin xyz="0 0 0" rpy="0 0 0"/>
-        <parent link="world"/>
-        <child link="link_0"/>
-    </joint>
     <link name="link_0">
         <visual>
@@ -33,5 +27,5 @@
     <link name="link_2">
         <visual>
-            <origin xyz="0.0 0.0 0.0" rpy="0 0 ${-M_PI/2}"/>
+            <origin xyz="0.0 0.0 0.0" rpy="0 0 0"/>
             <geometry>
                 <mesh filename="package://robot_description/meshes/link_2.stl" />
@@ -40,5 +34,5 @@
     </link>
     <joint name="joint_2" type="revolute">
-        <origin xyz="0.0 -0.12 0.0" rpy="${-M_PI/2} 0 0"/>
+        <origin xyz="0.0 -0.12 0.0" rpy="0 ${-M_PI/2} ${-M_PI/2}"/>
         <parent link="link_1"/>
         <child link="link_2"/>
@@ -48,5 +42,5 @@
     <link name="link_3">
         <visual>
-            <origin xyz="0.0 0.0 0.0" rpy="0 0 ${-M_PI/2}"/>
+            <origin xyz="0.0 0.0 0.0" rpy="0 0 0"/>
             <geometry>
                 <mesh filename="package://robot_description/meshes/link_3.stl" />
@@ -55,5 +49,5 @@
     </link>
     <joint name="joint_3" type="revolute">
-        <origin xyz="0.0 -0.25 0.1" rpy="0 0 ${-M_PI/2}"/>
+        <origin xyz="0.25 0.0 0.1" rpy="0 0 0"/>
         <parent link="link_2"/>
         <child link="link_3"/>
@@ -70,5 +64,5 @@
     </link>
     <joint name="joint_end_effector" type="fixed">
-        <origin xyz="0.0 -0.28 0.0" rpy="${M_PI/2} 0 0"/>
+        <origin xyz="0.28 0.0 0.0" rpy="${M_PI/2} 0 ${M_PI/2}"/>
         <parent link="link_3"/>
         <child link="end_effector"/>
