Commit message: update

File: src/robot_description/urdf/my-robot.urdf (robot description, URDF)
Before this commit: robot robot, 3 links, 2 joints
Links:
- added link end_effector; visual mesh filename=package://robot_description/meshes/end_effector.stl
- added link link_3; visual mesh filename=package://robot_description/meshes/link_3.stl
Joints:
- added joint joint_3: type revolute, parent link_2, child link_3, origin xyz=0.25 0.0 0.1 rpy=0 0 0, axis 0.0 0.0 1.0, limit lower=-3.14159 upper=3.14159 effort=1000.0 velocity=1000.0
- added joint joint_end_effector: type fixed, parent link_3, child end_effector, origin xyz=0.28 0.0 0.0 rpy=1.570795 0 1.570795
